File: Avionics Power Regulation Board/Avionics Power Regulation Board Subscale/Avionics Power Regulation Board Subscale.kicad_pcb (KiCad board)
At the start: 2 copper layers, 101.8 x 59.5 mm, 14 parts, among them J1 Conn_01x04_Socket, J2 Conn_01x06_Socket, J3 Conn_01x06_Socket, J4 Conn_01x08_Socket, U1 SC0917

Commit message: Small PCB Edits
Parts:
- added H2: MountingHole, MountingHole:MountingHole_2.1mm, F.Cu at (137.5, 95.9)
- added J5: Conn_01x05_Socket, Connector_PinSocket_2.54mm:PinSocket_1x05_P2.54mm_Vertical, F.Cu at (168.1, 41.4)
- J2: value Conn_01x06_Socket -> Conn_01x07_Socket
Connections:
- J2 pad 7: (no net) -> unconnected-(J2-Pin_7-Pad7)
