File: Avionics Power Regulation Board/Avionics Power Regulation Board.kicad_pcb (KiCad board)
At the start: 2 copper layers, 127.4 x 80.5 mm, 58 parts, among them J1 Conn_01x05_Socket, Q1 NMOS, Q2 NMOS, Q3 NMOS, SW1 SW_Push, U1 LM2576HVS-5, U2 BQ76920PW, U4 TPS61085DGK

Commit message: Fixed PMOS
Parts:
- removed D4, D5, D6: D, Diode_THT:D_DO-41_SOD81_P10.16mm_Horizontal
- moved D3 18.9 mm to (205.1, 83.7), turned to 90 degrees
- moved RSNS1 10.7 mm to (193.0, 64.5), turned to 90 degrees
- moved R9 1.85 mm to (201.3, 82.7)
Connections:
- Q1 pad 1: Net-(D3-K) -> Net-(Q1-Pad1)
- Q1 pad 3: Net-(D3-A) -> Net-(Q1-Pad3)
- Q2 pad 1: Net-(D4-A) -> Net-(D3-A)
- Q3 pad 1: Net-(D3-K) -> Net-(Q1-Pad1)
- Q3 pad 2: Net-(D5-K) -> Net-(D3-K)
- Q3 pad 3: GNDREF -> /Battery Monitor System/BAT -
- R4 pad 2: Net-(D3-A) -> Net-(Q1-Pad3)
- R6 pad 1: Net-(D3-A) -> Net-(Q1-Pad3)
- R8 pad 1: GNDREF -> /Battery Monitor System/BAT -
- R8 pad 2: Net-(D5-K) -> Net-(D3-K)
- R9 pad 1: Net-(D5-K) -> Net-(D3-K)
- R9 pad 2: Net-(D4-A) -> Net-(D3-A)
- RSNS1 pad 2: Net-(D3-A) -> Net-(Q1-Pad3)
Routing:
- net GNDREF: track 98.4 -> 66.0 mm, vias 4 -> 5
- net Net-(D3-K): track 43.7 -> 16.0 mm, vias 2 -> 0
- net Net-(D4-A): track 25.8 -> 0.00 mm, vias 1 -> 0
- net Net-(D5-K): track 20.8 -> 0.00 mm
- net Net-(Q1-Pad1): track 0.00 -> 18.3 mm
- net Net-(Q1-Pad3): track 0.00 -> 11.8 mm
- net /Battery Monitor System/BAT -: track 0.00 -> 9.39 mm
- net /Battery Monitor System/CHG: track 34.3 -> 31.4 mm
- net Net-(D3-A): track 27.6 -> 25.3 mm

Commit message: Fixed
Parts:
- removed the G*** at (124.0, 95.9)
- added G***: LOGO, AIAA Logo 2:AIAA Logo, B.Cu at (124.5, 81.9)
- added REF**: KiCad-Logo2_12mm_SilkScreen, Symbol:KiCad-Logo2_12mm_SilkScreen, B.Cu at (124.5, 113.8)
- Q1, Q3: footprint BS170:TO92 -> BS170_2:TO92
- Q2: value NMOS -> PMOS; footprint BS170:TO92 -> BS170_2:TO92
- moved G*** 0.23 mm to (124.1, 95.7)
- moved Q2 0.15 mm to (190.5, 73.7)
Connections:
- Q2 pad 2: /Battery Monitor System/CHG -> GNDREF
- Q2 pad 3: GNDREF -> /Battery Monitor System/CHG
Routing:
- net /Battery Monitor System/CHG: track 31.4 -> 32.1 mm
