File: Avionics Power Regulation Board/Avionics Instrumentation and Microcontroller/Avionics Instrumentation and Microcontroller Board.kicad_sch (KiCad schematic)
At the start: 19 parts, among them J1 Conn_01x04_Socket, J2 Conn_01x07_Socket, J3 Conn_01x06_Socket, J4 Conn_01x08_Socket, J5 Conn_01x05_Socket, J6 Conn_02x07_Odd_Even, J7 Micro_SD_Card_Det1, U1 SC0917

Commit message: Small Changes
Parts:
- removed J7: Micro_SD_Card_Det1, Connector_Card:microSD_HC_Hirose_DM3D-SF, symbol Connector:Micro_SD_Card_Det1
- added H12, H13: MountingHole, MountingHole:MountingHole_2.1mm, symbol Mechanical:MountingHole
- added J7: Conn_01x09_Socket, Connector_PinSocket_2.54mm:PinSocket_1x09_P2.54mm_Vertical, symbol Connector:Conn_01x09_Socket

Commit message: more changes
Parts:
- added H14: MountingHole, MountingHole:MountingHole_2.1mm, symbol Mechanical:MountingHole
Connections:
- net GNDREF: now also J1.4 (Pin_4), J2.3 (Pin_3), J3.6 (Pin_6), J4.2 (Pin_2), J5.1 (Pin_1), J7.2 (Pin_2), U1.A (USB_SHIELD), U1.B (USB_SHIELD), U1.C (USB_SHIELD), U1.D (USB_SHIELD)
- net 3.3V: now reaches J2.1 (Pin_1)
- net 3.3V: now also J1.1 (Pin_1), J3.1 (Pin_1), J4.1 (Pin_1), J7.1 (Pin_1), U1.36 (3V3_OUT)
- net Vin: now reaches U1.39 (VSYS)
- net Vin: now also J5.2 (Pin_2)
Other:
- note added: "Mounting Holes"
- moved on the sheet: H2, J5
